File: KiCad/WSON_driver.sch (KiCad schematic (older format))
At the start: 33 parts, among them K1 TIANBO-HJR-4102-L, Q2 PMOS_DGS, Q3 Q_NMOS_DGS, Q4 Q_NMOS_DGS, U4 LM25085SD_NOPB

Commit message: Latest schematics, all footprints except LED.
Parts:
- removed C12: Cout, symbol Device:CP1
- removed D5: D_Schottky, symbol Device:D_Schottky
- removed K1: TIANBO-HJR-4102-L, Relay_THT:Relay_SPDT_HJR-4102, symbol Relay:TIANBO-HJR-4102-L
- removed Q2: PMOS_DGS, symbol Device:Q_PMOS_DGS
- removed Q3, Q4: Q_NMOS_DGS, symbol Device:Q_NMOS_DGS
- added C12: Cout, Flashlight:CAP_10TPE47MAZB, symbol 10TPE47MAZB:10TPE47MAZB
- added D5: Driver_Schottky, Flashlight:TO-263-2, symbol Flashlight:Driver_Schottky
- added H5, H6: BMS_mnt, MountingHole:MountingHole_2.2mm_M2_Pad, symbol Mechanical:MountingHole
- added K1: HFD4-24-SR, Flashlight:HFD4024S, symbol HFD4_024-S:HFD4-24-SR
- added Q2: CSD25402Q3A, Flashlight:TRANS_CSD25402Q3A, symbol CSD25402Q3A:CSD25402Q3A
- added Q3, Q4: Q_NMOS_GSD, Package_TO_SOT_SMD:SOT-23_Handsoldering, symbol Device:Q_NMOS_GSD
- C11, C15, C16, C17: footprint (none) -> Capacitor_SMD:C_0805_2012Metric_Pad1.18x1.45mm_HandSolder
- C13, C18: footprint (none) -> Capacitor_SMD:C_0402_1005Metric_Pad0.74x0.62mm_HandSolder
- D6: value D -> D_flyback; footprint (none) -> Flashlight:D_SMAG
- H1, H2, H3, H4: footprint (none) -> MountingHole:MountingHole_2.5mm_Pad_Via
- L1: footprint (none) -> Flashlight:IHLP4040DZER2R2M01
- R11, R13, R16, R17, R19, R22: footprint (none) -> Resistor_SMD:R_0402_1005Metric_Pad0.72x0.64mm_HandSolder
- R12: footprint (none) -> Resistor_SMD:R_0805_2012Metric_Pad1.20x1.40mm_HandSolder
- R14, R18, R20, TH2: footprint (none) -> Resistor_SMD:R_0603_1608Metric_Pad0.98x0.95mm_HandSolder
- R15: footprint (none) -> Flashlight:TyoHM-SMF-3W
- R21: footprint (none) -> Flashlight:VZ067TL1B
- R9: footprint (none) -> Flashlight:R_1508_Wide
- U4: footprint SDA08A -> Flashlight:LM25085SD&slash_NOPB
Connections:
- wire segments 94 -> 84
Other:
- moved on the sheet: C11, C13, H1, H3, H4, L1, R11, R12
