File: KiCad/Flashlight.sch (KiCad schematic (older format))
At the start: 41 parts, among them J1 Screw_Terminal_01x02, J2 Conn_01x06_Female, J3 XT60PW-F, J4 Conn_01x06, Q1 PMOS_DGS, SW1 SW_DP3T, SW2 SW_Push, SW3 SW_SPST, U1 AMS1117-5.0, U2 PIC16F716-ISO, U3 LM60BIM3, Y1 Crystal

Commit message: Removed screw terminal, power input selection and ferrite bead filter.
Parts:
- removed C2: C, symbol Device:C
- removed FB1: Ferrite_Bead, symbol Device:Ferrite_Bead
- removed J1: Screw_Terminal_01x02, symbol Connector:Screw_Terminal_01x02
- removed SW1: SW_DP3T, symbol Switch:SW_DP3T
Connections:
- net labels removed: VTERM
- wire segments 114 -> 105
- no-connect marks 8 -> 7
Other:
- note removed: "Power source\nselection"
- moved on the sheet: C1, C3, D1, F1, Q1, R1, R2, TH1

Commit message: Latest schematics, all footprints except LED.
Parts:
- removed J3: XT60PW-F, AMASS_XT60PW-F, symbol XT60PW-F:XT60PW-F
- removed SW3: SW_SPST, symbol Switch:SW_SPST
- removed TH1: Thermistor NTC, symbol Device:Thermistor
- added C2: C, Capacitor_SMD:C_0402_1005Metric_Pad0.74x0.62mm_HandSolder, symbol Device:C
- added J3: XT30PW-F, Flashlight:XT30PWF, symbol XT30PW-F:XT30PW-F
- added R10, R23: R, Resistor_SMD:R_0402_1005Metric_Pad0.72x0.64mm_HandSolder, symbol Device:R
- added S1: SS-12D06L5, Flashlight:SS12D06L5, symbol SS-12D06L5:SS-12D06L5
- added SW1: SW_SPST, Flashlight:DSIC01LSGET, symbol Switch:SW_SPST
- added TP4: LED+, TestPoint:TestPoint_Pad_D2.0mm, symbol Connector:TestPoint
- C1, C4, C5: footprint (none) -> Capacitor_SMD:C_0603_1608Metric_Pad1.08x0.95mm_HandSolder
- C10, C3, C7, C8, C9: footprint (none) -> Capacitor_SMD:C_0402_1005Metric_Pad0.74x0.62mm_HandSolder
- C6: footprint (none) -> Capacitor_SMD:C_1210_3225Metric_Pad1.33x2.70mm_HandSolder
- D1: footprint (none) -> Package_TO_SOT_SMD:SOT-23_Handsoldering
- D2: footprint (none) -> Diode_SMD:D_SOD-323_HandSoldering
- D3, D4: footprint (none) -> LED_SMD:LED_0603_1608Metric_Pad1.05x0.95mm_HandSolder
- F1: value Fuse -> Fuse_PWR; footprint (none) -> Fuse:Fuse_1206_3216Metric_Pad1.42x1.75mm_HandSolder
- F2: value Fuse -> Fuse_LED; footprint (none) -> Fuse:Fuse_1206_3216Metric_Pad1.42x1.75mm_HandSolder
- J2: value Conn_01x06_Female -> LED
- J4: value Conn_01x06 -> ICSP 1x6; footprint (none) -> Flashlight:B6B-EH-A
- Q1: value PMOS_DGS -> PMOS_Vin; footprint (none) -> Package_SO:SOP-8-1EP_4.57x4.57mm_P1.27mm_EP4.57x4.45mm_ThermalVias
- R1: footprint (none) -> Resistor_SMD:R_0603_1608Metric_Pad0.98x0.95mm_HandSolder
- R2: value R -> 10k; footprint (none) -> Resistor_SMD:R_0402_1005Metric_Pad0.72x0.64mm_HandSolder
- R3, R4, R5, R6, R7, R8: footprint (none) -> Resistor_SMD:R_0402_1005Metric_Pad0.72x0.64mm_HandSolder
- SW2: footprint (none) -> Flashlight:SW_TS-1187A-B-A-B
- TP1: value TestPoint -> 5V; footprint (none) -> TestPoint:TestPoint_Pad_D2.0mm
- TP2: value TestPoint -> VDD; footprint (none) -> TestPoint:TestPoint_Pad_D2.0mm
- TP3: value TestPoint -> GND; footprint (none) -> TestPoint:TestPoint_Pad_D2.0mm
- U2: footprint (none) -> Flashlight:SOIC127P1030X265-18N
- U3: footprint MF03A -> Flashlight:LM60BIM3
- Y1: footprint (none) -> Flashlight:Crystal_SMD_3225-4Pin_3.2x2.5mm_HandSoldering
Connections:
- net labels added: ENABLE_DCDC
- wire segments 105 -> 118
- no-connect marks 7 -> 6
Other:
- note added: "Analog input"
- note removed: "100"
- note removed: "Inrush current\nlimit"
- moved on the sheet: C1, C10, C3, C4, C5, C6, C7, C8, C9, D1, D2, D3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

Commit message: Finished routing the first version of a PCB. WSON is out of stock so new driver was used.
Parts:
- removed J2: LED, symbol Connector:Conn_01x06_Female
- removed Q1: PMOS_Vin, Package_SO:SOP-8-1EP_4.57x4.57mm_P1.27mm_EP4.57x4.45mm_ThermalVias, symbol Device:Q_PMOS_DGS
- added J2: XHP90, Flashlight:XHP90, symbol Flashlight:XHP90
- added Q1: PMOS_Vin, Flashlight:YJS4407A, symbol Flashlight:YJS4407A
- J3: footprint Flashlight:XT30PWF -> Flashlight:AMASS_XT30PW-F
Connections:
- wire segments 118 -> 123
Changed lines of the file:
@@
 S 6800 1150 1350 650
 U 61784D48
-F0 "WSON_LED_driver" 50
-F1 "WSON_driver.sch" 50
+F0 "WSSOP_LED_driver" 50
+F1 "WSSOP_driver.sch" 50
 $EndSheet
 Text Notes 3500 1100 0    50   ~ 0
@@
 Wire Wire Line
 	9500 1500 9450 1500
-$Comp
-L Connector:Conn_01x06_Female J2
-U 1 1 61779D34
-P 10500 1400
-F 0 "J2" H 10528 1376 50  0000 L CNN
-F 1 "LED" H 10050 950 50  0000 L CNN
-F 2 "" H 10500 1400 50  0001 C CNN
-F 3 "~" H 10500 1400 50  0001 C CNN
-	1    10500 1400
-	1    0    0    -1
-$EndComp
 Wire Wire Line
 	10300 1200 10200 1200
@@
 P 1200 2950
 F 0 "C5" V 1350 2850 50  0000 C CNN
-F 1 "C" V 1361 2950 50  0000 C CNN
+F 1 "C" V 1361 2950 50  0001 C CNN
 F 2 "Capacitor_SMD:C_0603_1608Metric_Pad1.08x0.95mm_HandSolder" H 1238 2800 50  0001 C CNN
 F 3 "~" H 1200 2950 50  0001 C CNN
@@
 Wire Wire Line
 	4050 1400 3900 1400
-$Comp
-L Device:Q_PMOS_DGS Q1
-U 1 1 616E4D53
-P 3700 1500
-F 0 "Q1" V 4000 1550 50  0000 L CNN
-F 1 "PMOS_Vin" V 3905 1455 50  0000 L CNN
-F 2 "Package_SO:SOP-8-1EP_4.57x4.57mm_P1.27mm_EP4.57x4.45mm_ThermalVias" H 3900 1600 50  0001 C CNN
-F 3 "~" H 3700 1500 50  0001 C CNN
-	1    3700 1500
-	0    -1   -1   0
-$EndComp
 Wire Wire Line
 	3700 1750 3700 1700
@@
 F 0 "J3" H 2550 1150 50  0000 R CNN
 F 1 "XT30PW-F" H 2700 1650 50  0000 R CNN
-F 2 "Flashlight:XT30PWF" H 2750 1550 50  0001 L CNN
+F 2 "Flashlight:AMASS_XT30PW-F" H 2750 1550 50  0001 L CNN
 F 3 "https://www.tme.eu/Document/ce4077e36b79046da520ca73227e15de/XT30PW%20SPEC.pdf" H 2750 1450 50  0001 L CNN
 F 4 "Socket; DC supply; XT30; female; PIN:2; on PCBs; THT; Colour: yellow" H 2750 1350 50  0001 L CNN "Description"
@@
 Connection ~ 2150 1350
 Connection ~ 1300 1350
+$Comp
+L Flashlight:XHP90 J2
+U 1 1 61DC20C9
+P 10500 1400
+F 0 "J2" H 10528 1376 50  0000 L CNN
+F 1 "XHP90" H 10528 1285 50  0000 L CNN
+F 2 "Flashlight:XHP90" H 10500 1400 50  0001 C CNN
+F 3 "~" H 10500 1400 50  0001 C CNN
+	1    10500 1400
+	1    0    0    -1
+$EndComp
+$Comp
+L Flashlight:YJS4407A Q1
+U 1 1 61E5E62D
+P 3700 1500
+F 0 "Q1" V 4050 1500 50  0000 C CNN
+F 1 "PMOS_Vin" V 3950 1400 50  0000 C CNN
+F 2 "Flashlight:YJS4407A" H 3900 1600 50  0001 C CNN
+F 3 "~" H 3700 1500 50  0001 C CNN
+	1    3700 1500
+	0    -1   -1   0
+$EndComp
+Wire Wire Line
+	3500 1300 3500 1400
+Connection ~ 3500 1400
+Wire Wire Line
+	3500 1400 3500 1500
+Connection ~ 3500 1500
+Wire Wire Line
+	3500 1500 3500 1600
+Wire Wire Line
+	3900 1600 3900 1500
+Connection ~ 3900 1400
+Connection ~ 3900 1500
+Wire Wire Line
+	3900 1500 3900 1400
 $EndSCHEMATC
